File: motor-control-spi.sch (KiCad schematic (older format))
At the start: 29 parts, among them J1 Motor2, J2 PWR, J3 Motor1, J4 SPI, U1 AMS1117-5.0, U2 AMS1117-3.3, U3 L293D, U4 L293D, U5 MCP23S08-xP

Commit message: Added support libraries
Other:
- note added: "DECOUPLING CAPACITORS:"
Changed lines of the file:
@@
 Wire Wire Line
 	5530 2240 5670 2240
+Text Notes 1050 2210 0    59   ~ 12
+DECOUPLING CAPACITORS:
 $EndSCHEMATC
